File: ECAD/PCBs/OH_Specific/Backlighting_Type A/ECM DISP PANEL/ECM DISP PANEL.kicad_sch (KiCad schematic)
At the start: 89 parts, among them J1 BL IN, J2 BL OUT, J3 ECM JETT, SW1 ECM JETT

Commit message: Manufacturing File Update #3
COMM
DEFOG
ECM DISP
ECS
ELEC
EXT LT
FCS
FIRE TEST
FUEL
GEN TIE
HUD
Parts:
- removed H1, H2, H3, H4: MountingHole, MountingHole:MountingHole_4.5mm_Pad, symbol Mechanical:MountingHole
Changed lines of the file:
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@@
     (pin "4")
-  )
-  (symbol (lib_id "Mechanical:MountingHole") (at 195.58 19.05 0) (unit 1)
-    (in_bom yes) (on_board yes)
-    (property "Reference" "H1" (id 0) (at 198.12 17.8816 0)
-      (effects (font (size 1.27 1.27)) (justify left))
-    )
-    (property "Value" "MountingHole" (id 1) (at 198.12 20.193 0)
-      (effects (font (size 1.27 1.27)) (justify left))
-    )
-    (property "Footprint" "MountingHole:MountingHole_4.5mm_Pad" (id 2) (at 195.58 19.05 0)
-      (effects (font (size 1.27 1.27)) hide)
-    )
-    (property "Datasheet" "~" (id 3) (at 195.58 19.05 0)
-      (effects (font (size 1.27 1.27)) hide)
-    )
-  )
-  (symbol (lib_id "Mechanical:MountingHole") (at 195.58 24.13 0) (unit 1)
-    (in_bom yes) (on_board yes)
-    (property "Reference" "H2" (id 0) (at 198.12 22.9616 0)
-      (effects (font (size 1.27 1.27)) (justify left))
-    )
-    (property "Value" "MountingHole" (id 1) (at 198.12 25.273 0)
-      (effects (font (size 1.27 1.27)) (justify left))
-    )
-    (property "Footprint" "MountingHole:MountingHole_4.5mm_Pad" (id 2) (at 195.58 24.13 0)
-      (effects (font (size 1.27 1.27)) hide)
-    )
-    (property "Datasheet" "~" (id 3) (at 195.58 24.13 0)
-      (effects (font (size 1.27 1.27)) hide)
-    )
-  )
-  (symbol (lib_id "Mechanical:MountingHole") (at 195.58 29.21 0) (unit 1)
-    (in_bom yes) (on_board yes)
-    (property "Reference" "H3" (id 0) (at 198.12 28.0416 0)
-      (effects (font (size 1.27 1.27)) (justify left))
-    )
-    (property "Value" "MountingHole" (id 1) (at 198.12 30.353 0)
-      (effects (font (size 1.27 1.27)) (justify left))
-    )
-    (property "Footprint" "MountingHole:MountingHole_4.5mm_Pad" (id 2) (at 195.58 29.21 0)
-      (effects (font (size 1.27 1.27)) hide)
-    )
-    (property "Datasheet" "~" (id 3) (at 195.58 29.21 0)
-      (effects (font (size 1.27 1.27)) hide)
-    )
-  )
-  (symbol (lib_id "Mechanical:MountingHole") (at 195.58 34.29 0) (unit 1)
-    (in_bom yes) (on_board yes)
-    (property "Reference" "H4" (id 0) (at 198.12 33.1216 0)
-      (effects (font (size 1.27 1.27)) (justify left))
-    )
-    (property "Value" "MountingHole" (id 1) (at 198.12 35.433 0)
-      (effects (font (size 1.27 1.27)) (justify left))
-    )
-    (property "Footprint" "MountingHole:MountingHole_4.5mm_Pad" (id 2) (at 195.58 34.29 0)
-      (effects (font (size 1.27 1.27)) hide)
-    )
-    (property "Datasheet" "~" (id 3) (at 195.58 34.29 0)
-      (effects (font (size 1.27 1.27)) hide)
-    )
   )
   (sheet_instances
@@
       (reference "D79") (unit 1) (value "LED") (footprint "KiCAD Libraries:WS2812-2020")
     )
-    (path "/00000000-0000-0000-0000-000061642826"
-      (reference "H1") (unit 1) (value "MountingHole") (footprint "MountingHole:MountingHole_4.5mm_Pad")
-    )
-    (path "/00000000-0000-0000-0000-000061643121"
-      (reference "H2") (unit 1) (value "MountingHole") (footprint "MountingHole:MountingHole_4.5mm_Pad")
-    )
-    (path "/00000000-0000-0000-0000-0000616433c3"
-      (reference "H3") (unit 1) (value "MountingHole") (footprint "MountingHole:MountingHole_4.5mm_Pad")
-    )
-    (path "/00000000-0000-0000-0000-000061643571"
-      (reference "H4") (unit 1) (value "MountingHole") (footprint "MountingHole:MountingHole_4.5mm_Pad")
-    )
     (path "/00000000-0000-0000-0000-00005fd9ce4a"
