File: ECAD/PCBs/ABSIS/ABSIS_ALE/ABSIS_ALE.kicad_pcb (KiCad board)
At the start: 2 copper layers, 36 x 51 mm, 16 parts, among them J1 BUS IN, J2 BUS OUT, J3 I/O #1, J4 I/O #2, J5 GND, J6 ACC PWR, U1 MAX487EESA+T

Commit message: ECAD Directory update.
Parts:
- C1: footprint Capacitor_SMD:C_0805_2012Metric -> OH_Footprints:C_0805_2012Metric
- J1, J2: footprint Connector_Molex:Molex_Mini-Fit_Jr_5566-06A2_2x03_P4.20mm_Vertical -> OH_Footprints:Molex_Mini-Fit_Jr_5566-06A2_2x03_P4.20mm_Vertical
- J3, J4: footprint Connector_PinHeader_2.54mm:PinHeader_2x06_P2.54mm_Vertical -> OH_Footprints:PinHeader_2x06_P2.54mm_Vertical
- J5: footprint Connector_PinHeader_2.54mm:PinHeader_1x06_P2.54mm_Vertical -> OH_Footprints:PinHeader_1x06_P2.54mm_Vertical
- J6: footprint Connector_PinHeader_2.54mm:PinHeader_2x02_P2.54mm_Vertical -> OH_Footprints:PinHeader_2x02_P2.54mm_Vertical
- XU1: footprint Package_DIP:DIP-24_W15.24mm_Socket -> OH_Footprints:DIP-24_W15.24mm_Socket
Connections:
- net /~D10_A10 renamed /~{D10_A10}
- net /~D5 renamed /~{D5}
- net /~D6_A7 renamed /~{D6_A7}
- net /~D9_A9 renamed /~{D9_A9}
- net /~SCL_D3 renamed /~{SCL_D3}
Other:
- net class Default removed
- board text added: "~{10/ A10}"
- board text added: "~{D3}"
- board text added: "~{D6/ A7}"
- board text added: "~{D8/ A8}"
- board text added: "~{D9/ A9}"
- board text removed: "~10/ A10"
- board text removed: "~D3"
- board text removed: "~D6/ A7"
- board text removed: "~D8/ A8"
- board text removed: "~D9/ A9"
