File: ECAD/PCBs/ABSIS/ABSIS_ATX Power Supply Unit/ABSIS_ATX Power Supply Unit.kicad_pcb (KiCad board)
At the start: 4 copper layers, 144.4 x 71.1 mm, 45 parts, among them J1 I/O, J10 MEGA BUS 7, J11 MEGA BUS 8, J12 5V Accessory 1, J13 5V Accessory 2, J14 5V Accessory 3, J15 5V Accessory 4, J16 5V Accessory 5, J17 5V Accessory 6, J18 5V Accessory 7, J19 5V Accessory 8, J2 ATX-24, J20 12V Accessory 1, J21 12V Accessory 2, J22 12V Accessory 3, J23 12V Accessory 4, J24 12V Accessory 5, J25 PCIE IN 2, J26 PCIE IN 1, J28 EXTERNAL 5V IN, J29 BUTTKICKER AMP, J3 ABSIS BACKLIGHT, J30 EXTERNAL 12V IN, J4 MEGA BUS 1, J5 MEGA BUS 2, J6 MEGA BUS 3, J7 MEGA BUS 4, J8 MEGA BUS 5, J9 MEGA BUS 6

Commit message: Huge ECAD push
Parts:
- J25, J26: footprint Connector_Molex:Molex_Mini-Fit_Jr_5566-06A_2x03_P4.20mm_Vertical -> OH_Footprints:Molex_Mini-Fit_Jr_5566-06A_2x03_P4.20mm_Vertical
- moved J26 8.33 mm to (50.6, 62.5), turned to -90 degrees
- moved J25 5.38 mm to (50.6, 79.7), turned to -90 degrees
- moved J29 2.42 mm to (45.1, 98.9)
- moved J30 2.42 mm to (45.1, 111.8)
Other:
- board text added: "ABSIS ATX POWER SUPPLY UNIT"
- board text added: "REV 6"
- board text removed: "ABSIS ATX POWER DISTRIBUTION"
- board text removed: "REV 5"
