File: ECAD/PCBs/ABSIS/ABSIS_Mega/ABSIS_Mega.kicad_pcb (KiCad board)
At the start: 2 copper layers, 99.1 x 53.3 mm, 31 parts, among them J1 BUS IN, J2 BUS OUT, J3 DIGITAL #1, J4 ANALOG I/O, J5 DIGITAL #2, J6 DIGITAL #3, J7 ACC PWR, P1 Digital, P2 Power, P3 Analog, P4 Analog, P5 PWM, P6 PWM, P7 Communication, U1 MAX487EESA+T

Commit message: ECAD Directory update.
Other:
- net class Default removed
- board text added: "~{10}"
- board text added: "~{11}"
- board text added: "~{12}"
- board text added: "~{13}"
- board text added: "~{3}"
- board text added: "~{4}"
- board text added: "~{5}"
- board text added: "~{6}"
- board text added: "~{7}"
- board text added: "~{8}"
- board text added: "~{9}"
- board text removed: "~10"
- board text removed: "~11"
- board text removed: "~12"
- board text removed: "~13"
- board text removed: "~3"
- board text removed: "~4"
- board text removed: "~5"
- board text removed: "~6"
- board text removed: "~7"
- board text removed: "~8"
- board text removed: "~9"
