File: ECAD/PCBs/Backlight PCBs/Backlighting_Type A/ANT SEL PANEL/ANT SEL PANEL.kicad_pcb (KiCad board)
At the start: 2 copper layers, 85.2 x 43.2 mm, 30 parts, among them J1 Conn_01x04_Female, J2 Conn_01x04_Female

Commit message: Huge ECAD push
Parts:
- ?: renamed from G1; value LOGO -> (none); footprint Kicad Footprint Files:100SpxToggle -> OH_Footprints:100SP1_Toggle_Silkscreen
- ?: renamed from G2; value LOGO -> (none)
- ?: renamed from G3; value LOGO -> (none); footprint OH KiCAD_Libraries:OH_LOGO_37.7mm_5.9mm -> OH_Footprints:OH_LOGO_37.7mm_5.9mm
- CC-NC-SA_18mm_x_3.5mm: footprint OH_General:CC-NC-SA_18mm_x_3.5mm -> OH_Footprints:CC-NC-SA_18mm_x_3.5mm
- moved ? 1.45 mm to (126.5, 76.7)
Other:
- board text added: "ANT SEL PANEL Version 2.2 www.openhornet.com"
- board text removed: "ANT SEL Panel Backlight Designed by L.Walker"
- board text removed: "Version 2.1"
