File: ECAD/PCBs/Backlight PCBs/Backlighting_Type A/APU PANEL/APU PANEL.kicad_pcb (KiCad board)
At the start: 2 copper layers, 48.1 x 115.6 mm, 46 parts, among them J1 Conn_01x04_Female, J2 Conn_01x04_Female

Commit message: Huge ECAD push
Parts:
- renumbered G1 to ?, G4 to ?, G3 to ?, G2 to ?
Other:
- board text added: "APU PANEL Version: 2.4 www.openhornet.com"
- board text removed: "APU Panel Backlight Designed by L. Walker"
- board text removed: "Version 2.3"
Changed lines of the file:
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@@
     (at 90.97772 94.21876)
     (attr through_hole board_only exclude_from_pos_files exclude_from_bom)
-    (fp_text reference "G1" (at 0 10.1) (layer "F.SilkS") hide
+    (fp_text reference "" (at 0 10.1) (layer "F.SilkS") hide
       (effects (font (size 1.524 1.524) (thickness 0.3)))
     )
@@
     (at 101.7016 153.06802)
     (attr through_hole board_only exclude_from_pos_files exclude_from_bom)
-    (fp_text reference "G4" (at 0 10.1) (layer "F.SilkS") hide
+    (fp_text reference "" (at 0 10.1) (layer "F.SilkS") hide
       (effects (font (size 1.524 1.524) (thickness 0.3)))
     )
@@
     (at 91.45 130.95 180)
     (attr through_hole board_only exclude_from_pos_files exclude_from_bom)
-    (fp_text reference "G3" (at 0 0) (layer "B.SilkS") hide
+    (fp_text reference "" (at 0 0) (layer "B.SilkS") hide
       (effects (font (size 1.524 1.524) (thickness 0.3)) (justify mirror))
     )
@@
     (at 92.80906 119.82958 180)
     (attr through_hole board_only exclude_from_pos_files exclude_from_bom)
-    (fp_text reference "G2" (at 0 0) (layer "B.SilkS") hide
+    (fp_text reference "" (at 0 0) (layer "B.SilkS") hide
       (effects (font (size 1.524 1.524) (thickness 0.3)) (justify mirror))
     )
@@
     (effects (font (size 1.5 1.5) (thickness 0.3)) (justify mirror))
   )
-  (gr_text "APU Panel Backlight\nDesigned by L. Walker" (at 90.88882 111.9124) (layer "B.SilkS")
+  (gr_text "APU PANEL\nVersion: 2.4\n\nwww.openhornet.com" (at 92.202 110.744) (layer "B.SilkS")
     (effects (font (size 1 1) (thickness 0.15)) (justify mirror))
   )
@@
     (effects (font (size 1 1) (thickness 0.15)) (justify mirror))
   )
-  (gr_text "POWER REQUIREMENTS:\nVOLTAGE: 5V DC\nLEDS: 20\nCURRENT: 1.2A\nWATTAGE: 6.0W" (at 99.3 78.25) (layer "B.SilkS")
+  (gr_text "POWER REQUIREMENTS:\nVOLTAGE: 5V DC\nLEDS: 20\nCURRENT: 1.2A\nWATTAGE: 6.0W" (at 97.79 76.2) (layer "B.SilkS")
     (effects (font (size 1 1) (thickness 0.15)) (justify left mirror))
   )
@@
     (effects (font (size 1 1) (thickness 0.15)) (justify mirror))
   )
-  (gr_text "Version 2.3" (at 77.55 71.8) (layer "B.SilkS")
-    (effects (font (size 1 1) (thickness 0.15)) (justify mirror))
-  )
