File: ECAD/PCBs/Backlight PCBs/Backlighting_Type A/AV COOL PANEL/AV COOL PANEL.kicad_pcb (KiCad board)
At the start: 2 copper layers, 44.5 x 81.8 mm, 23 parts, among them J1 Conn_01x04_Female, J2 Conn_01x04_Female

Commit message: Huge ECAD push
Parts:
- ?: renamed from G***; footprint OH_General:CC-BY-NC-SA-Small -> OH_Footprints:CC-BY-NC-SA-Small
- ?: renamed from G***; footprint OH_General:OH_LOGO_ONLY_11x6mm -> OH_Footprints:OH_LOGO_ONLY_11x6mm
Other:
- board text added: "AV COOL PANEL Version 2.2 www.openhornet.com"
- board text removed: "AV COOL Panel Backlight Designed by L. Walker"
- board text removed: "Version 2.1"
