File: ECAD/PCBs/Backlight PCBs/Backlighting_Type A/CAUTION LIGHTS PANEL/CAUTION LIGHTS PANEL.kicad_pcb (KiCad board)
At the start: 2 copper layers, 81.9 x 39.8 mm, 59 parts, among them J1 Conn_01x04_Female, J2 Conn_01x04_Female

Commit message: Huge ECAD push
Parts:
- G***: footprint OH_General:OH_LOGO_37.7mm_5.9mm -> OH_Footprints:OH_LOGO_37.7mm_5.9mm
- G***: footprint OH_General:CC-BY-NC-SA-Small -> OH_Footprints:CC-BY-NC-SA-Small
Other:
- board text added: "CAUTION LIGHTS PANEL Version 2.0 www.openhornet.com"
- board text removed: "Caution Lights Panel Designed by L. Walker"
- board text removed: "Version 2.0"
