File: ECAD/PCBs/Backlight PCBs/Backlighting_Type A/HYD ISO PANEL/HYD ISO PANEL.kicad_pcb (KiCad board)
At the start: 2 copper layers, 104.3 x 38.9 mm, 50 parts, among them J1 Conn_01x04_Female, J2 Conn_01x04_Female

Commit message: Huge ECAD push
Other:
- board text added: "HYD ISO PANEL Version: 2.3 www.openhornet.com"
- board text removed: "HYD ISO Panel Backlight Designed by L.Walker"
- board text removed: "Version 2.2"
Changed lines of the file:
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@@
     (property "Sheetfile" "PCB, HYD ISO PANEL.kicad_sch")
     (property "Sheetname" "")
-    (attr through_hole exclude_from_pos_files)
+    (attr through_hole exclude_from_pos_files exclude_from_bom)
     (fp_text reference "D25" (at 1.27 2.96 180) (layer "B.SilkS")
       (effects (font (size 1 1) (thickness 0.15)) (justify mirror))
@@
   (gr_line (start 163.2712 60.3504) (end 171.958 69.4436) (layer "Edge.Cuts") (width 0.05))
   (gr_line (start 67.7 92.7) (end 74 99.25) (layer "Edge.Cuts") (width 0.05))
-  (gr_text "Version 2.2" (at 165.9 87.9) (layer "B.SilkS")
-    (effects (font (size 1 1) (thickness 0.15)) (justify mirror))
-  )
   (gr_text "2" (at 136.779 87.122) (layer "B.SilkS")
     (effects (font (size 1 1) (thickness 0.15)) (justify mirror))
@@
     (effects (font (size 1 1) (thickness 0.15)) (justify left mirror))
   )
-  (gr_text "HYD ISO\nPanel Backlight\nDesigned by L.Walker" (at 97.075 65.025) (layer "B.SilkS")
-    (effects (font (size 1 1) (thickness 0.15)) (justify left mirror))
+  (gr_text "HYD ISO PANEL\nVersion: 2.3\nwww.openhornet.com" (at 92.202 65.024) (layer "B.SilkS")
+    (effects (font (size 1 1) (thickness 0.15)) (justify mirror))
   )
   (gr_text "READY" (at 135.5 63.15) (layer "B.SilkS")
