File: ECAD/PCBs/Backlight PCBs/Backlighting_Type A/INTR LT PANEL/INTR LT PANEL.kicad_pcb (KiCad board)
At the start: 2 copper layers, 138.9 x 83.9 mm, 90 parts, among them J1 Conn_01x04_Female, J2 Conn_01x04_Female

Commit message: Huge ECAD push
Other:
- board text added: "INTR LT PANEL Version 2.2 www.openhornet.com"
- board text removed: "INTR LT Panel Backlight Designed by L. Walker Updated by Exprezzo Ver. 2.1"
Changed lines of the file:
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@@
     (effects (font (size 1 1) (thickness 0.15)) (justify mirror))
   )
-  (gr_text "INTR LT Panel Backlight\nDesigned by L. Walker\nUpdated by Exprezzo\nVer. 2.1" (at 69.65 90.35) (layer "B.SilkS")
+  (gr_text "INTR LT PANEL\nVersion 2.2\nwww.openhornet.com" (at 59.944 75.692) (layer "B.SilkS")
+    (effects (font (size 1 1) (thickness 0.15)) (justify mirror))
+  )
+  (gr_text "POWER REQUIREMENTS:\nVOLTAGE: 5V DC\nLEDS: 53\nCURRENT: 3.18A\nWATTAGE: 15.9W" (at 67.564 87.63) (layer "B.SilkS")
     (effects (font (size 1 1) (thickness 0.15)) (justify left mirror))
   )
-  (gr_text "POWER REQUIREMENTS:\nVOLTAGE: 5V DC\nLEDS: 53\nCURRENT: 3.18A\nWATTAGE: 15.9W" (at 143.425 123.2) (layer "B.SilkS")
-    (effects (font (size 1 1) (thickness 0.15)) (justify left mirror))
-  )
