File: ECAD/PCBs/Functional PCBs/ifei/ifei.kicad_pcb (KiCad board)
At the start: 2 copper layers, 165.1 x 120.7 mm, 57 parts, among them J1 BL IN, J2 BL OUT, J3 INPUTS, SW1 MODE, SW2 QTY, SW3 UP, SW4 DOWN, SW5 ZONE, SW6 ET

Commit message: Huge ECAD push
Parts:
- D1, D10, D11, D12, D13, D14, D15, D16, D17, D18, D19, D2, D20, D21, D22, D23, D24, D25, D26, D27, D28, D29, D3, D30, D31, D32, D33, D34, D35, D36, D37, D38, D39, D4, D5, D6, D7, D8, D9: footprint KiCAD Libraries:WS2812-2020 -> OH_Footprints:WS2812-2020
- J1, J2: footprint Connector_Molex:Molex_Mini-Fit_Jr_5566-04A_2x02_P4.20mm_Vertical -> OH_Footprints:Molex_Mini-Fit_Jr_5566-04A_2x02_P4.20mm_Vertical
- SW1, SW2, SW3, SW4, SW5, SW6: footprint Button_Switch_THT:SW_TH_Tactile_Omron_B3F-10xx -> OH_Footprints:SW_TH_Tactile_Omron_B3F-10xx
Other:
- outline, holes or cut-outs redrawn
- net class Default removed
