File: ECAD/PCBs/Functional PCBs/util_photoswitch/util_photoswitch.kicad_pcb (KiCad board)
At the start: 2 copper layers, 10 x 17 mm, 4 parts, among them J1 Conn_01x03_Male, U1 OPB615

Commit message: Huge ECAD push
Other:
- net class Default removed
