File: ECAD/PCBs/Backlight PCBs/Backlighting_Type A/SPIN RCV PANEL/SPIN RCV PANEL.kicad_pcb (KiCad board)
At the start: 2 copper layers, 45.7 x 168.3 mm, 66 parts, among them J1 Conn_01x04_Female, J2 Conn_01x04_Female

Commit message: software update
Use of Arduino IDE and Platform IO.  Adjusted file structure to match.
Parts:
- moved G*** 3.98 mm to (252.6, 63.6)
Other:
- board text added: "SPIN RCV PANEL Version 2.2 www.openhornet.com"
- board text removed: "SPIN RCVRY"
- board text removed: "Spin Panel Backlight Designed by L. Walker"
- board text removed: "Version 2.1"
